Commit message: first commit

File: panda/panda.urdf (robot description, URDF)
Before this commit: robot panda, 12 links, 11 joints
Links:
- link panda_hand: geometry collision mesh filename=meshes/collision/hand.obj; visual mesh filename=meshes/collision/hand.obj
- link panda_leftfinger: geometry collision mesh filename=meshes/collision/finger.obj; visual mesh filename=meshes/collision/finger.obj
- link panda_link0: geometry collision mesh filename=meshes/collision/link0.obj; visual mesh filename=meshes/collision/link0.obj
- link panda_link1: geometry collision mesh filename=meshes/collision/link1.obj; visual mesh filename=meshes/collision/link1.obj
- link panda_link2: geometry collision mesh filename=meshes/collision/link2.obj; visual mesh filename=meshes/collision/link2.obj
- link panda_link3: geometry collision mesh filename=meshes/collision/link3.obj; visual mesh filename=meshes/collision/link3.obj
- link panda_link4: geometry collision mesh filename=meshes/collision/link4.obj; visual mesh filename=meshes/collision/link4.obj
- link panda_link5: geometry collision mesh filename=meshes/collision/link5.obj; visual mesh filename=meshes/collision/link5.obj
- link panda_link6: geometry collision mesh filename=meshes/collision/link6.obj; visual mesh filename=meshes/collision/link6.obj
- link panda_link7: geometry collision mesh filename=meshes/collision/link7.obj; visual mesh filename=meshes/collision/link7.obj
- link panda_rightfinger: geometry collision mesh filename=meshes/collision/finger.obj; visual mesh filename=meshes/collision/finger.obj

Commit message: update mesh and code

File: panda/panda.urdf (robot description, URDF)
Before this commit: robot panda, 12 links, 11 joints
Links:
- removed link panda_hand
- removed link panda_leftfinger
- removed link panda_rightfinger
- added link panda_link0_sc; collision cylinder length=0.03 radius=0.09; collision sphere radius=0.09
- added link panda_link1_sc; collision cylinder length=0.283 radius=0.09; collision sphere radius=0.09
- added link panda_link2_sc; collision cylinder length=0.12 radius=0.09; collision sphere radius=0.09
- added link panda_link3_sc; collision cylinder length=0.15 radius=0.09; collision sphere radius=0.09
- added link panda_link4_sc; collision cylinder length=0.12 radius=0.09; collision sphere radius=0.09
- added link panda_link5_sc; collision cylinder length=0.1 radius=0.09; collision cylinder length=0.14 radius=0.055
- added link panda_link6_sc; collision cylinder length=0.08 radius=0.08; collision sphere radius=0.08
- added link panda_link7_sc; collision cylinder length=0.01 radius=0.06; collision cylinder length=0.14 radius=0.07
- link panda_link0: geometry collision mesh filename=./meshes/collision/link0.stl; visual mesh filename=./meshes/visual/link0.dae
- link panda_link1: geometry collision mesh filename=./meshes/collision/link1.stl; visual mesh filename=./meshes/visual/link1.dae
- link panda_link2: geometry collision mesh filename=./meshes/collision/link2.stl; visual mesh filename=./meshes/visual/link2.dae
- link panda_link3: geometry collision mesh filename=./meshes/collision/link3.stl; visual mesh filename=./meshes/visual/link3.dae
- link panda_link4: geometry collision mesh filename=./meshes/collision/link4.stl; visual mesh filename=./meshes/visual/link4.dae
- link panda_link5: geometry collision mesh filename=./meshes/collision/link5.stl; visual mesh filename=./meshes/visual/link5.dae
- link panda_link6: geometry collision mesh filename=./meshes/collision/link6.stl; visual mesh filename=./meshes/visual/link6.dae
- link panda_link7: geometry collision mesh filename=./meshes/collision/link7.stl; visual mesh filename=./meshes/visual/link7.dae
Joints:
- removed joint panda_finger_joint1
- removed joint panda_finger_joint2
- removed joint panda_hand_joint
- added joint panda_link0_sc_joint: type fixed, parent panda_link0, child panda_link0_sc, origin rpy=0 0 0
- added joint panda_link1_sc_joint: type fixed, parent panda_link1, child panda_link1_sc, origin rpy=0 0 0
- added joint panda_link2_sc_joint: type fixed, parent panda_link2, child panda_link2_sc, origin rpy=0 0 0
- added joint panda_link3_sc_joint: type fixed, parent panda_link3, child panda_link3_sc, origin rpy=0 0 0
- added joint panda_link4_sc_joint: type fixed, parent panda_link4, child panda_link4_sc, origin rpy=0 0 0
- added joint panda_link5_sc_joint: type fixed, parent panda_link5, child panda_link5_sc, origin rpy=0 0 0
- added joint panda_link6_sc_joint: type fixed, parent panda_link6, child panda_link6_sc, origin rpy=0 0 0
- added joint panda_link7_sc_joint: type fixed, parent panda_link7, child panda_link7_sc, origin rpy=0 0 0.7853981633974483
- joint panda_joint1: limit lower=-2.9671 upper=2.9671 effort=87 velocity=2.1750 -> lower=-2.8973 upper=2.8973 effort=87.0 velocity=2.175
- joint panda_joint2: limit lower=-1.8326 upper=1.8326 effort=87 velocity=2.1750 -> lower=-1.7628 upper=1.7628 effort=87.0 velocity=2.175; origin xyz=0 0 0 rpy=-1.57079632679 0 0 -> xyz=0 0 0 rpy=-1.5707963267948966 0 0
- joint panda_joint3: limit lower=-2.9671 upper=2.9671 effort=87 velocity=2.1750 -> lower=-2.8973 upper=2.8973 effort=87.0 velocity=2.175; origin xyz=0 -0.316 0 rpy=1.57079632679 0 0 -> xyz=0 -0.316 0 rpy=1.5707963267948966 0 0
- joint panda_joint4: limit lower=-3.1416 upper=0.0 effort=87 velocity=2.1750 -> lower=-3.0718 upper=-0.0698 effort=87.0 velocity=2.175; origin xyz=0.0825 0 0 rpy=1.57079632679 0 0 -> xyz=0.0825 0 0 rpy=1.5707963267948966 0 0
- joint panda_joint5: limit lower=-2.9671 upper=2.9671 effort=12 velocity=2.6100 -> lower=-2.8973 upper=2.8973 effort=12.0 velocity=2.61; origin xyz=-0.0825 0.384 0 rpy=-1.57079632679 0 0 -> xyz=-0.0825 0.384 0 rpy=-1.5707963267948966 0 0
- joint panda_joint6: limit lower=-0.0873 upper=3.8223 effort=12 velocity=2.6100 -> lower=-0.0175 upper=3.7525 effort=12.0 velocity=2.61; origin xyz=0 0 0 rpy=1.57079632679 0 0 -> xyz=0 0 0 rpy=1.5707963267948966 0 0
- joint panda_joint7: limit lower=-2.9671 upper=2.9671 effort=12 velocity=2.6100 -> lower=-2.8973 upper=2.8973 effort=12.0 velocity=2.61; origin xyz=0.088 0 0 rpy=1.57079632679 0 0 -> xyz=0.088 0 0 rpy=1.5707963267948966 0 0
- joint panda_joint8: axis 0 0 0 -> (none)

Commit message: fix mesh

File: panda/panda.urdf (robot description, URDF)
Before this commit: robot panda, 17 links, 16 joints
Links:
- link panda_link0: geometry collision mesh filename=meshes/collision/link0.stl; visual mesh filename=meshes/visual/link0.dae
- link panda_link1: geometry collision mesh filename=meshes/collision/link1.stl; visual mesh filename=meshes/visual/link1.dae
- link panda_link2: geometry collision mesh filename=meshes/collision/link2.stl; visual mesh filename=meshes/visual/link2.dae
- link panda_link3: geometry collision mesh filename=meshes/collision/link3.stl; visual mesh filename=meshes/visual/link3.dae
- link panda_link4: geometry collision mesh filename=meshes/collision/link4.stl; visual mesh filename=meshes/visual/link4.dae
- link panda_link5: geometry collision mesh filename=meshes/collision/link5.stl; visual mesh filename=meshes/visual/link5.dae
- link panda_link6: geometry collision mesh filename=meshes/collision/link6.stl; visual mesh filename=meshes/visual/link6.dae
- link panda_link7: geometry collision mesh filename=meshes/collision/link7.stl; visual mesh filename=meshes/visual/link7.dae
